Commit message: updated urdf for joint limits

File: src/kanga_core/kanga_core_description/urdf/core_2026.urdf.xacro (robot description, xacro)
@@ -5,8 +5,28 @@
   <xacro:arg name="prefix" default=""/>
   <xacro:arg name="drivetrain_profile" default="drivetrain_2025"/>
+  <!-- Validate compatibility before trying to load the selected profile. -->
+  <xacro:unless value="${'$(arg drivetrain_profile)' == 'drivetrain_2025'}">
+    <xacro:property
+      name="unsupported_drivetrain_profile"
+      value="${xacro.fatal('core_2026 requires drivetrain_2025; got', '$(arg drivetrain_profile)')}"
+      lazy_eval="false"
+    />
+  </xacro:unless>
+  <!-- Keep Gazebo joint limits tied to the selected physical drivetrain
+       profile. Continuous wheel joints deliberately have no position bounds. -->
+  <xacro:property
+    name="drivetrain_config_path"
+    value="../config/drivetrains/$(arg drivetrain_profile).yaml"
+  />
+  <xacro:property
+    name="drivetrain_config"
+    value="${xacro.load_yaml(drivetrain_config_path)}"
+  />
   <xacro:include filename="core_2026_macro.urdf.xacro"/>
   <xacro:core_2026
     prefix="$(arg prefix)"
     drivetrain_profile="$(arg drivetrain_profile)"
+    wheel_joint_effort_limit_nm="${drivetrain_config.drivetrain.wheel_joint_effort_limit_nm}"
+    wheel_joint_velocity_limit_rad_s="${drivetrain_config.drivetrain.motor_velocity_limit_tps * 2.0 * pi / drivetrain_config.drivetrain.motor_revolutions_per_wheel_revolution}"
   />
 </robot>

File: src/kanga_core/kanga_core_description/urdf/core_2026_macro.urdf.xacro (robot description, xacro)
@@ -4,8 +4,10 @@
        Params:
        - prefix: optional name prefix to avoid link/joint collisions
-       - drivetrain_profile: compatible physical drivetrain profile -->
+       - drivetrain_profile: compatible physical drivetrain profile
+       - wheel_joint_effort_limit_nm: high simulation effort ceiling
+       - wheel_joint_velocity_limit_rad_s: profile-derived wheel speed limit -->
   <xacro:macro
     name="core_2026"
-    params="prefix:='' drivetrain_profile:='drivetrain_2025'"
+    params="wheel_joint_effort_limit_nm wheel_joint_velocity_limit_rad_s prefix:='' drivetrain_profile:='drivetrain_2025'"
   >
     <!-- core_2026 describes the physical 2026 core, which retained the 2025
@@ -175,5 +177,5 @@
       <child link="${prefix}wheel_fl"/>
       <axis xyz="0 0 1"/>
-      <limit effort="0" velocity="0"/>
+      <limit effort="${wheel_joint_effort_limit_nm}" velocity="${wheel_joint_velocity_limit_rad_s}"/>
     </joint>
     <link name="${prefix}wheel_bl">
@@ -204,5 +206,5 @@
       <child link="${prefix}wheel_bl"/>
       <axis xyz="0 0 1"/>
-      <limit effort="0" velocity="0"/>
+      <limit effort="${wheel_joint_effort_limit_nm}" velocity="${wheel_joint_velocity_limit_rad_s}"/>
     </joint>
     <!-- Physical articulation range; state mapping lives in kanga_core_microcontroller. -->
@@ -290,5 +292,5 @@
       <child link="${prefix}wheel_fr"/>
       <axis xyz="0 0 1"/>
-      <limit effort="0" velocity="0"/>
+      <limit effort="${wheel_joint_effort_limit_nm}" velocity="${wheel_joint_velocity_limit_rad_s}"/>
     </joint>
     <link name="${prefix}wheel_br">
@@ -319,5 +321,5 @@
       <child link="${prefix}wheel_br"/>
       <axis xyz="0 0 1"/>
-      <limit effort="0" velocity="0"/>
+      <limit effort="${wheel_joint_effort_limit_nm}" velocity="${wheel_joint_velocity_limit_rad_s}"/>
     </joint>
     <!-- Physical articulation range; state mapping lives in kanga_core_microcontroller. -->
