Commit message: simplified collision models, updated body pose and suspension kinematics

File: src/kanga_core/kanga_core_description/urdf/core_2026_macro.urdf.xacro (robot description, xacro)
@@ -42,8 +42,16 @@
         </material>
       </visual>
-      <collision>
-        <origin xyz="-0.0406693 -0 0" rpy="0 0 1.5708"/>
-        <geometry>
-          <mesh filename="package://kanga_core_description/meshes/core_2026/core.stl"/>
+      <!-- Simplified chassis envelope; detailed mesh remains visual-only. -->
+      <collision>
+        <origin xyz="0.03833 0 0.0614" rpy="0 0 0"/>
+        <geometry>
+          <box size="0.683 0.3822 0.1228"/>
+        </geometry>
+      </collision>
+      <!-- Rear LED/e-stop protrusions above the main chassis. -->
+      <collision>
+        <origin xyz="-0.24116 -0.00339 0.2147" rpy="0 0 0"/>
+        <geometry>
+          <box size="0.070 0.2583 0.1838"/>
         </geometry>
       </collision>
@@ -57,8 +65,9 @@
         </material>
       </visual>
-      <collision>
-        <origin xyz="-0.0406693 -0 0" rpy="0 -0 1.5708"/>
-        <geometry>
-          <mesh filename="package://kanga_core_description/meshes/core_2026/antenna.stl"/>
+      <!-- Antenna mast cylinder derived from the visual-mesh envelope. -->
+      <collision>
+        <origin xyz="-0.24116 -0.19617 0.6196" rpy="0 0 0"/>
+        <geometry>
+          <cylinder radius="0.01275" length="1.131"/>
         </geometry>
       </collision>
@@ -105,8 +114,35 @@
         </material>
       </visual>
-      <collision>
-        <origin xyz="-0.189168 -0.0616 0.1911" rpy="-1.5708 1.5708 0"/>
-        <geometry>
-          <mesh filename="package://kanga_core_description/meshes/core_2026/left_suspension.stl"/>
+      <!-- Two straight suspension arms offset into the linkage plane. -->
+      <collision>
+        <origin xyz="0.139957 -0.166795 -0.0334" rpy="0 1.5708 -0.872665"/>
+        <geometry>
+          <cylinder radius="0.025" length="0.481171"/>
+        </geometry>
+      </collision>
+      <collision>
+        <origin xyz="-0.289321 -0.167040 -0.0334" rpy="0 1.5708 -2.617994"/>
+        <geometry>
+          <cylinder radius="0.025" length="0.698804"/>
+        </geometry>
+      </collision>
+      <!-- Shared suspension-arm pivot barrel. -->
+      <collision>
+        <origin xyz="0 -0.00286 0.0026" rpy="0 0 0"/>
+        <geometry>
+          <cylinder radius="0.026" length="0.112"/>
+        </geometry>
+      </collision>
+      <!-- Front and rear drivetrain housings. -->
+      <collision>
+        <origin xyz="0.279914 -0.333589 -0.090925" rpy="0 0 0"/>
+        <geometry>
+          <cylinder radius="0.065" length="0.2275"/>
+        </geometry>
+      </collision>
+      <collision>
+        <origin xyz="-0.578642 -0.334079 -0.090925" rpy="0 0 0"/>
+        <geometry>
+          <cylinder radius="0.065" length="0.2275"/>
         </geometry>
       </collision>
@@ -128,7 +164,7 @@
       </visual>
       <collision>
-        <origin xyz="0 -0 -0.05" rpy="-1.5708 0 0"/>
-        <geometry>
-          <mesh filename="package://kanga_core_description/meshes/core_2026/wheel_b.stl"/>
+        <origin xyz="0 0 0.04" rpy="0 0 0"/>
+        <geometry>
+          <cylinder radius="0.125" length="0.18"/>
         </geometry>
       </collision>
@@ -157,7 +193,7 @@
       </visual>
       <collision>
-        <origin xyz="0 0 -0.05" rpy="-1.5708 -0 0"/>
-        <geometry>
-          <mesh filename="package://kanga_core_description/meshes/core_2026/wheel_a.stl"/>
+        <origin xyz="0 0 0.04" rpy="0 0 0"/>
+        <geometry>
+          <cylinder radius="0.125" length="0.18"/>
         </geometry>
       </collision>
@@ -193,8 +229,35 @@
         </material>
       </visual>
-      <collision>
-        <origin xyz="0.189168 -0.0616 0.1911" rpy="-1.5708 -1.5708 0"/>
-        <geometry>
-          <mesh filename="package://kanga_core_description/meshes/core_2026/right_suspension.stl"/>
+      <!-- Two straight suspension arms offset into the linkage plane. -->
+      <collision>
+        <origin xyz="-0.139957 -0.166795 -0.0334" rpy="0 1.5708 -2.268927"/>
+        <geometry>
+          <cylinder radius="0.025" length="0.481150"/>
+        </geometry>
+      </collision>
+      <collision>
+        <origin xyz="0.289321 -0.167040 -0.0334" rpy="0 1.5708 -0.523599"/>
+        <geometry>
+          <cylinder radius="0.025" length="0.698789"/>
+        </geometry>
+      </collision>
+      <!-- Shared suspension-arm pivot barrel. -->
+      <collision>
+        <origin xyz="0 -0.00286 0.0026" rpy="0 0 0"/>
+        <geometry>
+          <cylinder radius="0.026" length="0.112"/>
+        </geometry>
+      </collision>
+      <!-- Front and rear drivetrain housings. -->
+      <collision>
+        <origin xyz="-0.279914 -0.333589 -0.090925" rpy="0 0 0"/>
+        <geometry>
+          <cylinder radius="0.065" length="0.2275"/>
+        </geometry>
+      </collision>
+      <collision>
+        <origin xyz="0.578642 -0.334079 -0.090925" rpy="0 0 0"/>
+        <geometry>
+          <cylinder radius="0.065" length="0.2275"/>
         </geometry>
       </collision>
@@ -216,7 +279,7 @@
       </visual>
       <collision>
-        <origin xyz="0 0 -0.05" rpy="-1.5708 -0 0"/>
-        <geometry>
-          <mesh filename="package://kanga_core_description/meshes/core_2026/wheel_a.stl"/>
+        <origin xyz="0 0 0.04" rpy="0 0 0"/>
+        <geometry>
+          <cylinder radius="0.125" length="0.18"/>
         </geometry>
       </collision>
@@ -245,7 +308,7 @@
       </visual>
       <collision>
-        <origin xyz="0 0 -0.05" rpy="-1.5708 0 0"/>
-        <geometry>
-          <mesh filename="package://kanga_core_description/meshes/core_2026/wheel_b.stl"/>
+        <origin xyz="0 0 0.04" rpy="0 0 0"/>
+        <geometry>
+          <cylinder radius="0.125" length="0.18"/>
         </geometry>
       </collision>
@@ -281,8 +344,9 @@
         </material>
       </visual>
-      <collision>
-        <origin xyz="-0 -0.0766 0.260486" rpy="-1.5708 -0 0"/>
-        <geometry>
-          <mesh filename="package://kanga_core_description/meshes/core_2026/diff_bar.stl"/>
+      <!-- Differential bar simplified to its rectangular envelope. -->
+      <collision>
+        <origin xyz="0 0.0015 -0.00026" rpy="0 0 0"/>
+        <geometry>
+          <box size="0.4055 0.033 0.0625"/>
         </geometry>
       </collision>

Commit message: wheel spin direction fisx + bug fix

File: src/kanga_core/kanga_core_description/urdf/core_2026_macro.urdf.xacro (robot description, xacro)
@@ -291,5 +291,7 @@
       <parent link="${prefix}right_suspension"/>
       <child link="${prefix}wheel_fr"/>
-      <axis xyz="0 0 1"/>
+      <!-- The mirrored right-suspension frame reverses local Z. Use -Z so
+           positive joint velocity means rover-forward on every wheel. -->
+      <axis xyz="0 0 -1"/>
       <limit effort="${wheel_joint_effort_limit_nm}" velocity="${wheel_joint_velocity_limit_rad_s}"/>
     </joint>
@@ -320,5 +322,6 @@
       <parent link="${prefix}right_suspension"/>
       <child link="${prefix}wheel_br"/>
-      <axis xyz="0 0 1"/>
+      <!-- Match the positive-forward wheel convention used by drive feedback. -->
+      <axis xyz="0 0 -1"/>
       <limit effort="${wheel_joint_effort_limit_nm}" velocity="${wheel_joint_velocity_limit_rad_s}"/>
     </joint>

Commit message: updated visualisation

File: src/kanga_core/kanga_core_description/urdf/core_2026_macro.urdf.xacro (robot description, xacro)
@@ -176,5 +176,5 @@
       <parent link="${prefix}left_suspension"/>
       <child link="${prefix}wheel_fl"/>
-      <axis xyz="0 0 1"/>
+      <axis xyz="0 0 -1"/>
       <limit effort="${wheel_joint_effort_limit_nm}" velocity="${wheel_joint_velocity_limit_rad_s}"/>
     </joint>
@@ -205,5 +205,5 @@
       <parent link="${prefix}left_suspension"/>
       <child link="${prefix}wheel_bl"/>
-      <axis xyz="0 0 1"/>
+      <axis xyz="0 0 -1"/>
       <limit effort="${wheel_joint_effort_limit_nm}" velocity="${wheel_joint_velocity_limit_rad_s}"/>
     </joint>
@@ -291,7 +291,7 @@
       <parent link="${prefix}right_suspension"/>
       <child link="${prefix}wheel_fr"/>
-      <!-- The mirrored right-suspension frame reverses local Z. Use -Z so
+      <!-- The mirrored right-suspension frame reverses local Z. Use +Z so
            positive joint velocity means rover-forward on every wheel. -->
-      <axis xyz="0 0 -1"/>
+      <axis xyz="0 0 1"/>
       <limit effort="${wheel_joint_effort_limit_nm}" velocity="${wheel_joint_velocity_limit_rad_s}"/>
     </joint>
@@ -323,5 +323,5 @@
       <child link="${prefix}wheel_br"/>
       <!-- Match the positive-forward wheel convention used by drive feedback. -->
-      <axis xyz="0 0 -1"/>
+      <axis xyz="0 0 1"/>
       <limit effort="${wheel_joint_effort_limit_nm}" velocity="${wheel_joint_velocity_limit_rad_s}"/>
     </joint>

Commit message: Developmenet of a sim for the core system. should act as a drop in replacement for the core of the rover with physics based suspension linkage

File: src/kanga_core/kanga_core_description/urdf/core_2026_macro.urdf.xacro (robot description, xacro)
@@ -6,8 +6,9 @@
        - drivetrain_profile: compatible physical drivetrain profile
        - wheel_joint_effort_limit_nm: high simulation effort ceiling
-       - wheel_joint_velocity_limit_rad_s: profile-derived wheel speed limit -->
+       - wheel_joint_velocity_limit_rad_s: profile-derived wheel speed limit
+       - passive_joint_*: finite simulation limits; they do not command hardware -->
   <xacro:macro
     name="core_2026"
-    params="wheel_joint_effort_limit_nm wheel_joint_velocity_limit_rad_s prefix:='' drivetrain_profile:='drivetrain_2025'"
+    params="wheel_joint_effort_limit_nm wheel_joint_velocity_limit_rad_s prefix:='' drivetrain_profile:='drivetrain_2025' wheel_joint_damping_nm_s_rad:=0.0 passive_joint_effort_limit_nm:=500.0 passive_joint_velocity_limit_rad_s:=2.0 passive_joint_damping_nm_s_rad:=0.0"
   >
     <!-- core_2026 describes the physical 2026 core, which retained the 2025
@@ -178,4 +179,5 @@
       <axis xyz="0 0 -1"/>
       <limit effort="${wheel_joint_effort_limit_nm}" velocity="${wheel_joint_velocity_limit_rad_s}"/>
+      <dynamics damping="${wheel_joint_damping_nm_s_rad}" friction="0"/>
     </joint>
     <link name="${prefix}wheel_bl">
@@ -207,4 +209,5 @@
       <axis xyz="0 0 -1"/>
       <limit effort="${wheel_joint_effort_limit_nm}" velocity="${wheel_joint_velocity_limit_rad_s}"/>
+      <dynamics damping="${wheel_joint_damping_nm_s_rad}" friction="0"/>
     </joint>
     <!-- Physical articulation range; state mapping lives in kanga_core_microcontroller. -->
@@ -214,5 +217,6 @@
       <child link="${prefix}left_suspension"/>
       <axis xyz="0 0 1"/>
-      <limit effort="0" velocity="0" lower="-0.5235987755982988" upper="0.5235987755982988"/>
+      <limit effort="${passive_joint_effort_limit_nm}" velocity="${passive_joint_velocity_limit_rad_s}" lower="-0.5235987755982988" upper="0.5235987755982988"/>
+      <dynamics damping="${passive_joint_damping_nm_s_rad}" friction="0"/>
     </joint>
     <link name="${prefix}right_suspension">
@@ -295,4 +299,5 @@
       <axis xyz="0 0 1"/>
       <limit effort="${wheel_joint_effort_limit_nm}" velocity="${wheel_joint_velocity_limit_rad_s}"/>
+      <dynamics damping="${wheel_joint_damping_nm_s_rad}" friction="0"/>
     </joint>
     <link name="${prefix}wheel_br">
@@ -325,4 +330,5 @@
       <axis xyz="0 0 1"/>
       <limit effort="${wheel_joint_effort_limit_nm}" velocity="${wheel_joint_velocity_limit_rad_s}"/>
+      <dynamics damping="${wheel_joint_damping_nm_s_rad}" friction="0"/>
     </joint>
     <!-- Physical articulation range; state mapping lives in kanga_core_microcontroller. -->
@@ -332,5 +338,6 @@
       <child link="${prefix}right_suspension"/>
       <axis xyz="0 0 1"/>
-      <limit effort="0" velocity="0" lower="-0.5235987755982988" upper="0.5235987755982988"/>
+      <limit effort="${passive_joint_effort_limit_nm}" velocity="${passive_joint_velocity_limit_rad_s}" lower="-0.5235987755982988" upper="0.5235987755982988"/>
+      <dynamics damping="${passive_joint_damping_nm_s_rad}" friction="0"/>
     </joint>
     <link name="${prefix}diff_bar">
@@ -363,5 +370,6 @@
       <child link="${prefix}diff_bar"/>
       <axis xyz="0 0 1"/>
-      <limit effort="0" velocity="0" lower="-1.2217304763960306" upper="1.2217304763960306"/>
+      <limit effort="${passive_joint_effort_limit_nm}" velocity="${passive_joint_velocity_limit_rad_s}" lower="-1.2217304763960306" upper="1.2217304763960306"/>
+      <dynamics damping="${passive_joint_damping_nm_s_rad}" friction="0"/>
     </joint>
   </xacro:macro>
